Commit message: fixing cadanarm, creat entity and $ paths
Signed-off-by: Dharini Dutia <dharini@openrobotics.org>

File: models/curiosity_path/urdf/right_wheel_group.xacro (robot description, xacro)
@@ -7,12 +7,12 @@
 					rpy="0 0 0"/>
 			<geometry>
-				<mesh filename="(find simulation)/models/curiosity_path/meshes/right_axis_jointfix_v2.dae" scale="${scale_XYZ} ${scale_XYZ} ${scale_XYZ}"/>
-			</geometry>
-		</collision>
-		<visual>
-			<origin xyz="0 0 0"
-					rpy="0 0 0"/>
-			<geometry>
-				<mesh filename="(find simulation)/models/curiosity_path/meshes/right_axis_jointfix_v2.dae" scale="${scale_XYZ} ${scale_XYZ} ${scale_XYZ}"/>
+				<mesh filename="$(find simulation)/models/curiosity_path/meshes/right_axis_jointfix_v2.dae" scale="${scale_XYZ} ${scale_XYZ} ${scale_XYZ}"/>
+			</geometry>
+		</collision>
+		<visual>
+			<origin xyz="0 0 0"
+					rpy="0 0 0"/>
+			<geometry>
+				<mesh filename="$(find simulation)/models/curiosity_path/meshes/right_axis_jointfix_v2.dae" scale="${scale_XYZ} ${scale_XYZ} ${scale_XYZ}"/>
 			</geometry>
 		</visual>
@@ -38,12 +38,12 @@
 					rpy="0 0 0"/>
 			<geometry>
-				<mesh filename="(find simulation)/models/curiosity_path/meshes/suspension_arm_F_R_fixed.dae" scale="${scale_XYZ} ${scale_XYZ} ${scale_XYZ}"/>
-			</geometry>
-		</collision>
-		<visual>
-			<origin xyz="0 0 0"
-					rpy="0 0 0"/>
-			<geometry>
-				<mesh filename="(find simulation)/models/curiosity_path/meshes/suspension_arm_F_R_fixed.dae" scale="${scale_XYZ} ${scale_XYZ} ${scale_XYZ}"/>
+				<mesh filename="$(find simulation)/models/curiosity_path/meshes/suspension_arm_F_R_fixed.dae" scale="${scale_XYZ} ${scale_XYZ} ${scale_XYZ}"/>
+			</geometry>
+		</collision>
+		<visual>
+			<origin xyz="0 0 0"
+					rpy="0 0 0"/>
+			<geometry>
+				<mesh filename="$(find simulation)/models/curiosity_path/meshes/suspension_arm_F_R_fixed.dae" scale="${scale_XYZ} ${scale_XYZ} ${scale_XYZ}"/>
 			</geometry>
 		</visual>
@@ -82,12 +82,12 @@
 					rpy="0 0 0"/>
 			<geometry>
-				<mesh filename="(find simulation)/models/curiosity_path/meshes/suspension_arm_B_R_fixed.dae" scale="${scale_XYZ} ${scale_XYZ} ${scale_XYZ}"/>
-			</geometry>
-		</collision>
-		<visual>
-			<origin xyz="0 0 0"
-					rpy="0 0 0"/>
-			<geometry>
-				<mesh filename="(find simulation)/models/curiosity_path/meshes/suspension_arm_B_R_fixed.dae" scale="${scale_XYZ} ${scale_XYZ} ${scale_XYZ}"/>
+				<mesh filename="$(find simulation)/models/curiosity_path/meshes/suspension_arm_B_R_fixed.dae" scale="${scale_XYZ} ${scale_XYZ} ${scale_XYZ}"/>
+			</geometry>
+		</collision>
+		<visual>
+			<origin xyz="0 0 0"
+					rpy="0 0 0"/>
+			<geometry>
+				<mesh filename="$(find simulation)/models/curiosity_path/meshes/suspension_arm_B_R_fixed.dae" scale="${scale_XYZ} ${scale_XYZ} ${scale_XYZ}"/>
 			</geometry>
 		</visual>
@@ -150,12 +150,12 @@
 					rpy="0 0 0"/>
 			<geometry>
-				<mesh filename="(find simulation)/models/curiosity_path/meshes/suspension_arm_B2_R_fixed.dae" scale="${scale_XYZ} ${scale_XYZ} ${scale_XYZ}"/>
-			</geometry>
-		</collision>
-		<visual>
-			<origin xyz="0 0 0"
-					rpy="0 0 0"/>
-			<geometry>
-				<mesh filename="(find simulation)/models/curiosity_path/meshes/suspension_arm_B2_R_fixed.dae" scale="${scale_XYZ} ${scale_XYZ} ${scale_XYZ}"/>
+				<mesh filename="$(find simulation)/models/curiosity_path/meshes/suspension_arm_B2_R_fixed.dae" scale="${scale_XYZ} ${scale_XYZ} ${scale_XYZ}"/>
+			</geometry>
+		</collision>
+		<visual>
+			<origin xyz="0 0 0"
+					rpy="0 0 0"/>
+			<geometry>
+				<mesh filename="$(find simulation)/models/curiosity_path/meshes/suspension_arm_B2_R_fixed.dae" scale="${scale_XYZ} ${scale_XYZ} ${scale_XYZ}"/>
 			</geometry>
 		</visual>
@@ -219,12 +219,12 @@
 					rpy="0 0 0"/>
 			<geometry>
-				<mesh filename="(find simulation)/models/curiosity_path/meshes/suspension_steer_F_R_fixed.dae" scale="${scale_XYZ} ${scale_XYZ} ${scale_XYZ}"/>
-			</geometry>
-		</collision>
-		<visual>
-			<origin xyz="0 0 0"
-					rpy="0 0 0"/>
-			<geometry>
-				<mesh filename="(find simulation)/models/curiosity_path/meshes/suspension_steer_F_R_fixed.dae" scale="${scale_XYZ} ${scale_XYZ} ${scale_XYZ}"/>
+				<mesh filename="$(find simulation)/models/curiosity_path/meshes/suspension_steer_F_R_fixed.dae" scale="${scale_XYZ} ${scale_XYZ} ${scale_XYZ}"/>
+			</geometry>
+		</collision>
+		<visual>
+			<origin xyz="0 0 0"
+					rpy="0 0 0"/>
+			<geometry>
+				<mesh filename="$(find simulation)/models/curiosity_path/meshes/suspension_steer_F_R_fixed.dae" scale="${scale_XYZ} ${scale_XYZ} ${scale_XYZ}"/>
 			</geometry>
 		</visual>
@@ -344,12 +344,12 @@
 					rpy="0 0 0"/>
 			<geometry>
-				<mesh filename="(find simulation)/models/curiosity_path/meshes/suspension_steer_B_R_fixed.dae" scale="${scale_XYZ} ${scale_XYZ} ${scale_XYZ}"/>
-			</geometry>
-		</collision>
-		<visual>
-			<origin xyz="0 0 0"
-					rpy="0 0 0"/>
-			<geometry>
-				<mesh filename="(find simulation)/models/curiosity_path/meshes/suspension_steer_B_R_fixed.dae" scale="${scale_XYZ} ${scale_XYZ} ${scale_XYZ}"/>
+				<mesh filename="$(find simulation)/models/curiosity_path/meshes/suspension_steer_B_R_fixed.dae" scale="${scale_XYZ} ${scale_XYZ} ${scale_XYZ}"/>
+			</geometry>
+		</collision>
+		<visual>
+			<origin xyz="0 0 0"
+					rpy="0 0 0"/>
+			<geometry>
+				<mesh filename="$(find simulation)/models/curiosity_path/meshes/suspension_steer_B_R_fixed.dae" scale="${scale_XYZ} ${scale_XYZ} ${scale_XYZ}"/>
 			</geometry>
 		</visual>

File: models/curiosity_path/urdf/sensor_mast.xacro (robot description, xacro)
@@ -31,5 +31,5 @@
 					rpy="0 0 0"/>
 			<geometry>
-				<mesh filename="(find simulation)/models/curiosity_path/meshes/mast_p_fixed.dae" scale="${scale_XYZ} ${scale_XYZ} ${scale_XYZ}"/>
+				<mesh filename="$(find simulation)/models/curiosity_path/meshes/mast_p_fixed.dae" scale="${scale_XYZ} ${scale_XYZ} ${scale_XYZ}"/>
 			</geometry>
 		</collision>
@@ -38,5 +38,5 @@
 					rpy="0 0 0"/>
 			<geometry>
-				<mesh filename="(find simulation)/models/curiosity_path/meshes/mast_p_fixed.dae" scale="${scale_XYZ} ${scale_XYZ} ${scale_XYZ}"/>
+				<mesh filename="$(find simulation)/models/curiosity_path/meshes/mast_p_fixed.dae" scale="${scale_XYZ} ${scale_XYZ} ${scale_XYZ}"/>
 			</geometry>
 		</visual>
@@ -99,5 +99,5 @@
 					rpy="0 0 0"/>
 			<geometry>
-				<mesh filename="(find simulation)/models/curiosity_path/meshes/mast_02_fixed.dae" scale="${scale_XYZ} ${scale_XYZ} ${scale_XYZ}"/>
+				<mesh filename="$(find simulation)/models/curiosity_path/meshes/mast_02_fixed.dae" scale="${scale_XYZ} ${scale_XYZ} ${scale_XYZ}"/>
 			</geometry>
 		</collision>
@@ -106,5 +106,5 @@
 					rpy="0 0 0"/>
 			<geometry>
-				<mesh filename="(find simulation)/models/curiosity_path/meshes/mast_02_fixed.dae" scale="${scale_XYZ} ${scale_XYZ} ${scale_XYZ}"/>
+				<mesh filename="$(find simulation)/models/curiosity_path/meshes/mast_02_fixed.dae" scale="${scale_XYZ} ${scale_XYZ} ${scale_XYZ}"/>
 			</geometry>
 		</visual>
@@ -167,5 +167,5 @@
 					rpy="0 0 0"/>
 			<geometry>
-				<mesh filename="(find simulation)/models/curiosity_path/meshes/mast_cameras.dae" scale="${scale_XYZ} ${scale_XYZ} ${scale_XYZ}"/>
+				<mesh filename="$(find simulation)/models/curiosity_path/meshes/mast_cameras.dae" scale="${scale_XYZ} ${scale_XYZ} ${scale_XYZ}"/>
 			</geometry>
 		</collision>
@@ -174,5 +174,5 @@
 					rpy="0 0 0"/>
 			<geometry>
-				<mesh filename="(find simulation)/models/curiosity_path/meshes/mast_cameras.dae" scale="${scale_XYZ} ${scale_XYZ} ${scale_XYZ}"/>
+				<mesh filename="$(find simulation)/models/curiosity_path/meshes/mast_cameras.dae" scale="${scale_XYZ} ${scale_XYZ} ${scale_XYZ}"/>
 			</geometry>
 		</visual>

File: models/curiosity_path/urdf/wheel.xacro (robot description, xacro)
@@ -15,5 +15,5 @@
 					rpy="0 0 0"/>
 			<geometry>
-				<mesh filename="(find simulation)/models/curiosity_path/meshes/wheel_fixed.dae" scale="${scale_XYZ} ${scale_XYZ} ${scale_XYZ}"/>
+				<mesh filename="$(find simulation)/models/curiosity_path/meshes/wheel_fixed.dae" scale="${scale_XYZ} ${scale_XYZ} ${scale_XYZ}"/>
 			</geometry>
 		</visual>

Commit message: collision meshes
Signed-off-by: Dharini Dutia <dharini@openrobotics.org>

File: models/canadarm/urdf/SSRMS_Canadarm2.urdf (robot description, URDF)
Before this commit: robot SSRMS_Canadarm2, 9 links, 8 joints
Links:
- link B1: geometry collision mesh filename=file:///$(find simulation)/models/canadarm/meshes/joint_com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 scale=1.0 1.0 1.0; visual mesh filename=file:///$(find simulation)/models/canadarm/meshes/joint_v3_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 scale=1.0 1.0 1.0
- link B2: geometry collision mesh filename=file:///$(find simulation)/models/canadarm/meshes/joint_com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 scale=1.0 1.0 1.0; visual mesh filename=file:///$(find simulation)/models/canadarm/meshes/joint_v3_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 scale=1.0 1.0 1.0
- link B3: geometry collision mesh filename=file:///$(find simulation)/models/canadarm/meshes/joint_com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 scale=1.0 1.0 1.0; collision mesh filename=file:///$(find simulation)/models/canadarm/meshes/joint_com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 scale=1.0 1.0 1.0
- link B4: geometry collision mesh filename=file:///$(find simulation)/models/canadarm/meshes/joint_com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 scale=1.0 1.0 1.0; collision mesh filename=file:///$(find simulation)/models/canadarm/meshes/link_join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 scale=1.0 1.0 1.0
- link B5: geometry collision mesh filename=file:///$(find simulation)/models/canadarm/meshes/joint_com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 scale=1.0 1.0 1.0; visual mesh filename=file:///$(find simulation)/models/canadarm/meshes/joint_v3_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 scale=1.0 1.0 1.0
- link B6: geometry collision mesh filename=file:///$(find simulation)/models/canadarm/meshes/joint_com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 scale=1.0 1.0 1.0; visual mesh filename=file:///$(find simulation)/models/canadarm/meshes/joint_v3_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 scale=1.0 1.0 1.0
- link Base_SSRMS: geometry collision mesh filename=file:///$(find simulation)/models/canadarm/meshes/ee.stl scale=1.0 1.0 1.0; visual mesh filename=file:///$(find simulation)/models/canadarm/meshes/ee.dae scale=1.0 1.0 1.0
- link EE_SSRMS: geometry collision mesh filename=file:///$(find simulation)/models/canadarm/meshes/ee.stl scale=1.0 1.0 1.0; visual mesh filename=file:///$(find simulation)/models/canadarm/meshes/ee.dae scale=1.0 1.0 1.0
