Commit message: Add Apollo 15 Lunar Roving Vehicle

File: models/curiosity_path/urdf/chassis.xacro (robot description, xacro)
@@ -4,7 +4,13 @@
     <!-- Used for fixing robot to Gazebo 'chassis' -->
 	<link name="base_footprint" />
-	<joint name="base_joint" type="fixed">
+	<link name="base_link" />
+	<joint name="base_footprint_to_link" type="fixed">
 		<parent link="base_footprint"/>
+		<child link="base_link"/>
+	</joint>
+	<joint name="base_to_chassis" type="fixed">
+		<parent link="base_link"/>
 		<child link="chassis"/>
+		<origin rpy="0 0 1.57" xyz="0 0 0"/>
 	</joint>
 	<link name='chassis'>
@@ -13,5 +19,5 @@
 					rpy="0 0 0"/>
 			<geometry>
-				<mesh filename="$(find simulation)/models/curiosity_path/meshes/chassis_full_fixed_glitch_v2.dae" scale="${scale_XYZ} ${scale_XYZ} ${scale_XYZ}"/>
+				<mesh filename="package://simulation/models/curiosity_path/meshes/chassis_full_fixed_glitch_v2.dae" scale="${scale_XYZ} ${scale_XYZ} ${scale_XYZ}"/>
 			</geometry>
 		</collision>
@@ -20,5 +26,5 @@
 					rpy="0 0 0"/>
 			<geometry>
-				<mesh filename="$(find simulation)/models/curiosity_path/meshes/chassis_full_fixed_glitch_v2.dae" scale="${scale_XYZ} ${scale_XYZ} ${scale_XYZ}"/>
+				<mesh filename="package://simulation/models/curiosity_path/meshes/chassis_full_fixed_glitch_v2.dae" scale="${scale_XYZ} ${scale_XYZ} ${scale_XYZ}"/>
 			</geometry>
 		</visual>

File: models/curiosity_path/urdf/sensor_mast.xacro (robot description, xacro)
@@ -31,5 +31,5 @@
 					rpy="0 0 0"/>
 			<geometry>
-				<mesh filename="$(find simulation)/models/curiosity_path/meshes/mast_p_fixed.dae" scale="${scale_XYZ} ${scale_XYZ} ${scale_XYZ}"/>
+				<mesh filename="package://simulation/models/curiosity_path/meshes/mast_p_fixed.dae" scale="${scale_XYZ} ${scale_XYZ} ${scale_XYZ}"/>
 			</geometry>
 		</collision>
@@ -38,5 +38,5 @@
 					rpy="0 0 0"/>
 			<geometry>
-				<mesh filename="$(find simulation)/models/curiosity_path/meshes/mast_p_fixed.dae" scale="${scale_XYZ} ${scale_XYZ} ${scale_XYZ}"/>
+				<mesh filename="package://simulation/models/curiosity_path/meshes/mast_p_fixed.dae" scale="${scale_XYZ} ${scale_XYZ} ${scale_XYZ}"/>
 			</geometry>
 		</visual>
@@ -99,5 +99,5 @@
 					rpy="0 0 0"/>
 			<geometry>
-				<mesh filename="$(find simulation)/models/curiosity_path/meshes/mast_02_fixed.dae" scale="${scale_XYZ} ${scale_XYZ} ${scale_XYZ}"/>
+				<mesh filename="package://simulation/models/curiosity_path/meshes/mast_02_fixed.dae" scale="${scale_XYZ} ${scale_XYZ} ${scale_XYZ}"/>
 			</geometry>
 		</collision>
@@ -106,5 +106,5 @@
 					rpy="0 0 0"/>
 			<geometry>
-				<mesh filename="$(find simulation)/models/curiosity_path/meshes/mast_02_fixed.dae" scale="${scale_XYZ} ${scale_XYZ} ${scale_XYZ}"/>
+				<mesh filename="package://simulation/models/curiosity_path/meshes/mast_02_fixed.dae" scale="${scale_XYZ} ${scale_XYZ} ${scale_XYZ}"/>
 			</geometry>
 		</visual>
@@ -167,5 +167,5 @@
 					rpy="0 0 0"/>
 			<geometry>
-				<mesh filename="$(find simulation)/models/curiosity_path/meshes/mast_cameras.dae" scale="${scale_XYZ} ${scale_XYZ} ${scale_XYZ}"/>
+				<mesh filename="package://simulation/models/curiosity_path/meshes/mast_cameras.dae" scale="${scale_XYZ} ${scale_XYZ} ${scale_XYZ}"/>
 			</geometry>
 		</collision>
@@ -174,5 +174,5 @@
 					rpy="0 0 0"/>
 			<geometry>
-				<mesh filename="$(find simulation)/models/curiosity_path/meshes/mast_cameras.dae" scale="${scale_XYZ} ${scale_XYZ} ${scale_XYZ}"/>
+				<mesh filename="package://simulation/models/curiosity_path/meshes/mast_cameras.dae" scale="${scale_XYZ} ${scale_XYZ} ${scale_XYZ}"/>
 			</geometry>
 		</visual>
@@ -232,4 +232,27 @@
         <origin xyz="0.13642 -0.218683 0.222314" rpy="0 0 ${-PI/2}"/>
     </joint>
+  	<link name="lidar_link">
+        <!-- Inertial for gazebo to take it into account, Put 1gr weight -->
+        <inertial>
+            <origin xyz="0 0 0" rpy="0 0 0"/>
+            <mass value="0.001" />
+            <inertia ixx="9.1875e-09" ixy="0.0" ixz="0.0" iyy="9.1875e-09" iyz="0.0" izz="1.378125e-08"/>
+        </inertial>
+		<visual>
+            <origin rpy="0.0 0 0" xyz="0 0 0"/>
+            <geometry>
+                <cylinder radius="0.05" length="0.02"/>
+            </geometry>
+            <material name="black"/>
+        </visual>
+	</link>
+    <gazebo reference="lidar_link">
+        <material>Gazebo/Black</material>
+    </gazebo>
+    <joint name="lidar_joint" type="fixed">
+        <parent link="mast_cameras"/>
+        <child link="lidar_link"/>
+        <origin xyz="0 0 0.325" rpy="0 0 ${-PI/2}"/>
+    </joint>
   </xacro:macro>
 </robot>
