Commit message: paths in xacro files
Signed-off-by: Dharini Dutia <dharini@openrobotics.org>

File: models/curiosity_path/urdf/arm.xacro (robot description, xacro)
@@ -31,12 +31,12 @@
 					rpy="0 0 0"/>
 			<geometry>
-				<mesh filename="package://mars_rover/meshes/arm_01_fixed.dae" scale="${scale_XYZ} ${scale_XYZ} ${scale_XYZ}"/>
-			</geometry>
-		</collision>
-		<visual>
-			<origin xyz="0 0 0"
-					rpy="0 0 0"/>
-			<geometry>
-				<mesh filename="package://mars_rover/meshes/arm_01_fixed.dae" scale="${scale_XYZ} ${scale_XYZ} ${scale_XYZ}"/>
+				<mesh filename="package://simulation/models/curiosity_path/meshes/arm_01_fixed.dae" scale="${scale_XYZ} ${scale_XYZ} ${scale_XYZ}"/>
+			</geometry>
+		</collision>
+		<visual>
+			<origin xyz="0 0 0"
+					rpy="0 0 0"/>
+			<geometry>
+				<mesh filename="package://simulation/models/curiosity_path/meshes/arm_01_fixed.dae" scale="${scale_XYZ} ${scale_XYZ} ${scale_XYZ}"/>
 			</geometry>
 		</visual>
@@ -99,12 +99,12 @@
 					rpy="0 0 0"/>
 			<geometry>
-				<mesh filename="package://mars_rover/meshes/arm_01_fixed.dae" scale="${scale_XYZ} ${scale_XYZ} ${scale_XYZ}"/>
-			</geometry>
-		</collision>
-		<visual>
-			<origin xyz="0 0 0"
-					rpy="0 0 0"/>
-			<geometry>
-				<mesh filename="package://mars_rover/meshes/arm_02_fixed.dae" scale="${scale_XYZ} ${scale_XYZ} ${scale_XYZ}"/>
+				<mesh filename="package://simulation/models/curiosity_path/meshes/arm_01_fixed.dae" scale="${scale_XYZ} ${scale_XYZ} ${scale_XYZ}"/>
+			</geometry>
+		</collision>
+		<visual>
+			<origin xyz="0 0 0"
+					rpy="0 0 0"/>
+			<geometry>
+				<mesh filename="package://simulation/models/curiosity_path/meshes/arm_02_fixed.dae" scale="${scale_XYZ} ${scale_XYZ} ${scale_XYZ}"/>
 			</geometry>
 		</visual>
@@ -167,12 +167,12 @@
 					rpy="0 0 0"/>
 			<geometry>
-				<mesh filename="package://mars_rover/meshes/arm_03_fixed.dae" scale="${scale_XYZ} ${scale_XYZ} ${scale_XYZ}"/>
-			</geometry>
-		</collision>
-		<visual>
-			<origin xyz="0 0 0"
-					rpy="0 0 0"/>
-			<geometry>
-				<mesh filename="package://mars_rover/meshes/arm_03_fixed.dae" scale="${scale_XYZ} ${scale_XYZ} ${scale_XYZ}"/>
+				<mesh filename="package://simulation/models/curiosity_path/meshes/arm_03_fixed.dae" scale="${scale_XYZ} ${scale_XYZ} ${scale_XYZ}"/>
+			</geometry>
+		</collision>
+		<visual>
+			<origin xyz="0 0 0"
+					rpy="0 0 0"/>
+			<geometry>
+				<mesh filename="package://simulation/models/curiosity_path/meshes/arm_03_fixed.dae" scale="${scale_XYZ} ${scale_XYZ} ${scale_XYZ}"/>
 			</geometry>
 		</visual>
@@ -235,12 +235,12 @@
 					rpy="0 0 0"/>
 			<geometry>
-				<mesh filename="package://mars_rover/meshes/arm_04_fixed.dae" scale="${scale_XYZ} ${scale_XYZ} ${scale_XYZ}"/>
-			</geometry>
-		</collision>
-		<visual>
-			<origin xyz="0 0 0"
-					rpy="0 0 0"/>
-			<geometry>
-				<mesh filename="package://mars_rover/meshes/arm_04_fixed.dae" scale="${scale_XYZ} ${scale_XYZ} ${scale_XYZ}"/>
+				<mesh filename="package://simulation/models/curiosity_path/meshes/arm_04_fixed.dae" scale="${scale_XYZ} ${scale_XYZ} ${scale_XYZ}"/>
+			</geometry>
+		</collision>
+		<visual>
+			<origin xyz="0 0 0"
+					rpy="0 0 0"/>
+			<geometry>
+				<mesh filename="package://simulation/models/curiosity_path/meshes/arm_04_fixed.dae" scale="${scale_XYZ} ${scale_XYZ} ${scale_XYZ}"/>
 			</geometry>
 		</visual>
@@ -303,12 +303,12 @@
 					rpy="0 0 0"/>
 			<geometry>
-				<mesh filename="package://mars_rover/meshes/arm_tools_fixed.dae" scale="${scale_XYZ} ${scale_XYZ} ${scale_XYZ}"/>
-			</geometry>
-		</collision>
-		<visual>
-			<origin xyz="0 0 0"
-					rpy="0 0 0"/>
-			<geometry>
-				<mesh filename="package://mars_rover/meshes/arm_tools_fixed.dae" scale="${scale_XYZ} ${scale_XYZ} ${scale_XYZ}"/>
+				<mesh filename="package://simulation/models/curiosity_path/meshes/arm_tools_fixed.dae" scale="${scale_XYZ} ${scale_XYZ} ${scale_XYZ}"/>
+			</geometry>
+		</collision>
+		<visual>
+			<origin xyz="0 0 0"
+					rpy="0 0 0"/>
+			<geometry>
+				<mesh filename="package://simulation/models/curiosity_path/meshes/arm_tools_fixed.dae" scale="${scale_XYZ} ${scale_XYZ} ${scale_XYZ}"/>
 			</geometry>
 		</visual>

File: models/curiosity_path/urdf/chassis.xacro (robot description, xacro)
@@ -13,5 +13,5 @@
 					rpy="0 0 0"/>
 			<geometry>
-				<mesh filename="/home/spaceros-user/src/spaceros_demo/install/mars_rover/share/mars_rover/meshes/chassis_full_fixed_glitch_v2.dae" scale="${scale_XYZ} ${scale_XYZ} ${scale_XYZ}"/>
+				<mesh filename="package://simulation/models/curiosity_path/meshes/chassis_full_fixed_glitch_v2.dae" scale="${scale_XYZ} ${scale_XYZ} ${scale_XYZ}"/>
 			</geometry>
 		</collision>
@@ -20,5 +20,5 @@
 					rpy="0 0 0"/>
 			<geometry>
-				<mesh filename="/home/spaceros-user/src/spaceros_demo/install/mars_rover/share/mars_rover/meshes/chassis_full_fixed_glitch_v2.dae" scale="${scale_XYZ} ${scale_XYZ} ${scale_XYZ}"/>
+				<mesh filename="package://simulation/models/curiosity_path/meshes/chassis_full_fixed_glitch_v2.dae" scale="${scale_XYZ} ${scale_XYZ} ${scale_XYZ}"/>
 			</geometry>
 		</visual>

File: models/curiosity_path/urdf/curiosity_mars_rover.xacro (robot description, xacro)
@@ -2,19 +2,19 @@
 <robot name="curiosity_mars_rover" xmlns:xacro="http://wiki.ros.org/xacro">
     <!-- Inertia matrices -->
-	<xacro:include filename="$(find mars_rover)/urdf/macros.xacro" />
+	<xacro:include filename="$(find simulation)/curiosity_path/urdf/macros.xacro" />
 	<!-- Robot constants and properties -->
-	<xacro:include filename="$(find mars_rover)/urdf/curiosity_mars_rover_properties.xacro" />
+	<xacro:include filename="$(find simulation)/curiosity_path/urdf/curiosity_mars_rover_properties.xacro" />
 	<!-- Gazebo aspects of the robot -->
-	<xacro:include filename="$(find mars_rover)/urdf/curiosity_mars_rover.gazebo" />
+	<xacro:include filename="$(find simulation)/curiosity_path/urdf/curiosity_mars_rover.gazebo" />
 	<!-- Chasis -->
-	<xacro:include filename="$(find mars_rover)/urdf/chassis.xacro" />
+	<xacro:include filename="$(find simulation)/curiosity_path/urdf/chassis.xacro" />
 	<!-- Wheel Groups -->
-	<xacro:include filename="$(find mars_rover)/urdf/wheel.xacro" />
-	<xacro:include filename="$(find mars_rover)/urdf/left_wheel_group.xacro" />
-	<xacro:include filename="$(find mars_rover)/urdf/right_wheel_group.xacro" />
+	<xacro:include filename="$(find simulation)/curiosity_path/urdf/wheel.xacro" />
+	<xacro:include filename="$(find simulation)/curiosity_path/urdf/left_wheel_group.xacro" />
+	<xacro:include filename="$(find simulation)/curiosity_path/urdf/right_wheel_group.xacro" />
 	<!-- Arm -->
-	<xacro:include filename="$(find mars_rover)/urdf/arm.xacro" />
+	<xacro:include filename="$(find simulation)/curiosity_path/urdf/arm.xacro" />
 	<!-- Sensor Mast -->
-	<xacro:include filename="$(find mars_rover)/urdf/sensor_mast.xacro" />
+	<xacro:include filename="$(find simulation)/curiosity_path/urdf/sensor_mast.xacro" />
 	<xacro:chassis_body/>
 	<xacro:left_wheel_tree/>

File: models/curiosity_path/urdf/curiosity_mars_rover.xacro.urdf (robot description, URDF)
Before this commit: robot curiosity_mars_rover, 49 links, 48 joints
Links:
- link arm_01: geometry collision mesh filename=package://simulation/models/curiosity_path/meshes/arm_01_fi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 scale=1.0 1.0 1.0; visual mesh filename=package://simulation/models/curiosity_path/meshes/arm_01_fi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 scale=1.0 1.0 1.0
- link arm_02: geometry collision mesh filename=package://simulation/models/curiosity_path/meshes/arm_01_fi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 scale=1.0 1.0 1.0; visual mesh filename=package://simulation/models/curiosity_path/meshes/arm_02_fi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 scale=1.0 1.0 1.0
- link arm_03: geometry collision mesh filename=package://simulation/models/curiosity_path/meshes/arm_03_fi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 scale=1.0 1.0 1.0; visual mesh filename=package://simulation/models/curiosity_path/meshes/arm_03_fi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 scale=1.0 1.0 1.0
- link arm_04: geometry collision mesh filename=package://simulation/models/curiosity_path/meshes/arm_04_fi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 scale=1.0 1.0 1.0; visual mesh filename=package://simulation/models/curiosity_path/meshes/arm_04_fi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 scale=1.0 1.0 1.0
- link arm_tools: geometry collision mesh filename=package://simulation/models/curiosity_path/meshes/arm_tools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 scale=1.0 1.0 1.0; visual mesh filename=package://simulation/models/curiosity_path/meshes/arm_tools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 scale=1.0 1.0 1.0
- link back_wheel_L: geometry collision cylinder length=0.39473 radius=0.242647; visual mesh filename=package://simulation/models/curiosity_path/meshes/wheel_fix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 scale=1.0 1.0 1.0
- link back_wheel_R: geometry collision cylinder length=0.39473 radius=0.242647; visual mesh filename=package://simulation/models/curiosity_path/meshes/wheel_fix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 scale=1.0 1.0 1.0
- link chassis: geometry collision mesh scale=1.0 1.0 1.0 uri=package://simulation/models/curiosity_path/meshes/chassis_f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; visual mesh filename=package://simulation/models/curiosity_path/meshes/chassis_f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 scale=1.0 1.0 1.0
- link front_wheel_L: geometry collision cylinder length=0.39473 radius=0.242647; visual mesh filename=package://simulation/models/curiosity_path/meshes/wheel_fix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 scale=1.0 1.0 1.0
- link front_wheel_R: geometry collision cylinder length=0.39473 radius=0.242647; visual mesh filename=package://simulation/models/curiosity_path/meshes/wheel_fix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 scale=1.0 1.0 1.0
- link left_axis: geometry collision mesh filename=package://simulation/models/curiosity_path/meshes/left_axis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 scale=1.0 1.0 1.0; visual mesh filename=package://simulation/models/curiosity_path/meshes/left_axis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 scale=1.0 1.0 1.0
- link mast_02: geometry collision mesh filename=package://simulation/models/curiosity_path/meshes/mast_02_f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 scale=1.0 1.0 1.0; visual mesh filename=package://simulation/models/curiosity_path/meshes/mast_02_f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 scale=1.0 1.0 1.0
- link mast_cameras: geometry collision mesh filename=package://simulation/models/curiosity_path/meshes/mast_came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 scale=1.0 1.0 1.0; visual mesh filename=package://simulation/models/curiosity_path/meshes/mast_came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 scale=1.0 1.0 1.0
- link mast_p: geometry collision mesh filename=package://simulation/models/curiosity_path/meshes/mast_p_fi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 scale=1.0 1.0 1.0; visual mesh filename=package://simulation/models/curiosity_path/meshes/mast_p_fi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 scale=1.0 1.0 1.0
- link middle_wheel_L: geometry collision cylinder length=0.39473 radius=0.242647; visual mesh filename=package://simulation/models/curiosity_path/meshes/wheel_fix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 scale=1.0 1.0 1.0
- link middle_wheel_R: geometry collision cylinder length=0.39473 radius=0.242647; visual mesh filename=package://simulation/models/curiosity_path/meshes/wheel_fix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 scale=1.0 1.0 1.0
- link right_axis: geometry collision mesh filename=package://simulation/models/curiosity_path/meshes/right_axi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 scale=1.0 1.0 1.0; visual mesh filename=package://simulation/models/curiosity_path/meshes/right_axi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 scale=1.0 1.0 1.0
- link suspension_arm_B2_L: geometry collision mesh filename=package://simulation/models/curiosity_path/meshes/suspensio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 scale=1.0 1.0 1.0; visual mesh filename=package://simulation/models/curiosity_path/meshes/suspensio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 scale=1.0 1.0 1.0
- link suspension_arm_B2_R: geometry collision mesh filename=package://simulation/models/curiosity_path/meshes/suspensio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 scale=1.0 1.0 1.0; visual mesh filename=package://simulation/models/curiosity_path/meshes/suspensio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 scale=1.0 1.0 1.0
- link suspension_arm_B_L: geometry collision mesh filename=package://simulation/models/curiosity_path/meshes/suspensio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 scale=1.0 1.0 1.0; visual mesh filename=package://simulation/models/curiosity_path/meshes/suspensio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 scale=1.0 1.0 1.0
- link suspension_arm_B_R: geometry collision mesh filename=package://simulation/models/curiosity_path/meshes/suspensio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 scale=1.0 1.0 1.0; visual mesh filename=package://simulation/models/curiosity_path/meshes/suspensio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 scale=1.0 1.0 1.0
- link suspension_arm_F_L: geometry collision mesh filename=package://simulation/models/curiosity_path/meshes/suspensio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 scale=1.0 1.0 1.0; visual mesh filename=package://simulation/models/curiosity_path/meshes/suspensio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 scale=1.0 1.0 1.0
- link suspension_arm_F_R: geometry collision mesh filename=package://simulation/models/curiosity_path/meshes/suspensio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 scale=1.0 1.0 1.0; visual mesh filename=package://simulation/models/curiosity_path/meshes/suspensio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 scale=1.0 1.0 1.0
- link suspension_steer_B_L: geometry collision mesh filename=package://simulation/models/curiosity_path/meshes/suspensio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 scale=1.0 1.0 1.0; visual mesh filename=package://simulation/models/curiosity_path/meshes/suspensio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 scale=1.0 1.0 1.0
- link suspension_steer_B_R: geometry collision mesh filename=package://simulation/models/curiosity_path/meshes/suspensio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 scale=1.0 1.0 1.0; visual mesh filename=package://simulation/models/curiosity_path/meshes/suspensio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 scale=1.0 1.0 1.0
- link suspension_steer_F_L: geometry collision mesh filename=package://simulation/models/curiosity_path/meshes/suspensio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 scale=1.0 1.0 1.0; visual mesh filename=package://simulation/models/curiosity_path/meshes/suspensio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 scale=1.0 1.0 1.0
- link suspension_steer_F_R: geometry collision mesh filename=package://simulation/models/curiosity_path/meshes/suspensio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 scale=1.0 1.0 1.0; visual mesh filename=package://simulation/models/curiosity_path/meshes/suspensio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 scale=1.0 1.0 1.0

File: models/curiosity_path/urdf/left_wheel_group.xacro (robot description, xacro)
@@ -7,12 +7,12 @@
 					rpy="0 0 0"/>
 			<geometry>
-				<mesh filename="/home/spaceros-user/src/spaceros_demo/install/mars_rover/share/mars_rover/meshes/left_axis_jointfix_v2.dae" scale="${scale_XYZ} ${scale_XYZ} ${scale_XYZ}"/>
-			</geometry>
-		</collision>
-		<visual>
-			<origin xyz="0 0 0"
-					rpy="0 0 0"/>
-			<geometry>
-				<mesh filename="/home/spaceros-user/src/spaceros_demo/install/mars_rover/share/mars_rover/meshes/left_axis_jointfix_v2.dae" scale="${scale_XYZ} ${scale_XYZ} ${scale_XYZ}"/>
+				<mesh filename="package://simulation/models/curiosity_path/meshes/left_axis_jointfix_v2.dae" scale="${scale_XYZ} ${scale_XYZ} ${scale_XYZ}"/>
+			</geometry>
+		</collision>
+		<visual>
+			<origin xyz="0 0 0"
+					rpy="0 0 0"/>
+			<geometry>
+				<mesh filename="package://simulation/models/curiosity_path/meshes/left_axis_jointfix_v2.dae" scale="${scale_XYZ} ${scale_XYZ} ${scale_XYZ}"/>
 			</geometry>
 		</visual>
@@ -38,12 +38,12 @@
 					rpy="0 0 0"/>
 			<geometry>
-				<mesh filename="/home/spaceros-user/src/spaceros_demo/install/mars_rover/share/mars_rover/meshes/suspension_arm_F_L_fixed.dae" scale="${scale_XYZ} ${scale_XYZ} ${scale_XYZ}"/>
-			</geometry>
-		</collision>
-		<visual>
-			<origin xyz="0 0 0"
-					rpy="0 0 0"/>
-			<geometry>
-				<mesh filename="/home/spaceros-user/src/spaceros_demo/install/mars_rover/share/mars_rover/meshes/suspension_arm_F_L_fixed.dae" scale="${scale_XYZ} ${scale_XYZ} ${scale_XYZ}"/>
+				<mesh filename="package://simulation/models/curiosity_path/meshes/suspension_arm_F_L_fixed.dae" scale="${scale_XYZ} ${scale_XYZ} ${scale_XYZ}"/>
+			</geometry>
+		</collision>
+		<visual>
+			<origin xyz="0 0 0"
+					rpy="0 0 0"/>
+			<geometry>
+				<mesh filename="package://simulation/models/curiosity_path/meshes/suspension_arm_F_L_fixed.dae" scale="${scale_XYZ} ${scale_XYZ} ${scale_XYZ}"/>
 			</geometry>
 		</visual>
@@ -82,12 +82,12 @@
 					rpy="0 0 0"/>
 			<geometry>
-				<mesh filename="/home/spaceros-user/src/spaceros_demo/install/mars_rover/share/mars_rover/meshes/suspension_arm_B_L_fixed.dae" scale="${scale_XYZ} ${scale_XYZ} ${scale_XYZ}"/>
-			</geometry>
-		</collision>
-		<visual>
-			<origin xyz="0 0 0"
-					rpy="0 0 0"/>
-			<geometry>
-				<mesh filename="/home/spaceros-user/src/spaceros_demo/install/mars_rover/share/mars_rover/meshes/suspension_arm_B_L_fixed.dae" scale="${scale_XYZ} ${scale_XYZ} ${scale_XYZ}"/>
+				<mesh filename="package://simulation/models/curiosity_path/meshes/suspension_arm_B_L_fixed.dae" scale="${scale_XYZ} ${scale_XYZ} ${scale_XYZ}"/>
+			</geometry>
+		</collision>
+		<visual>
+			<origin xyz="0 0 0"
+					rpy="0 0 0"/>
+			<geometry>
+				<mesh filename="package://simulation/models/curiosity_path/meshes/suspension_arm_B_L_fixed.dae" scale="${scale_XYZ} ${scale_XYZ} ${scale_XYZ}"/>
 			</geometry>
 		</visual>
@@ -150,12 +150,12 @@
 					rpy="0 0 0"/>
 			<geometry>
-				<mesh filename="/home/spaceros-user/src/spaceros_demo/install/mars_rover/share/mars_rover/meshes/suspension_arm_B2_L_fixed.dae" scale="${scale_XYZ} ${scale_XYZ} ${scale_XYZ}"/>
-			</geometry>
-		</collision>
-		<visual>
-			<origin xyz="0 0 0"
-					rpy="0 0 0"/>
-			<geometry>
-				<mesh filename="/home/spaceros-user/src/spaceros_demo/install/mars_rover/share/mars_rover/meshes/suspension_arm_B2_L_fixed.dae" scale="${scale_XYZ} ${scale_XYZ} ${scale_XYZ}"/>
+				<mesh filename="package://simulation/models/curiosity_path/meshes/suspension_arm_B2_L_fixed.dae" scale="${scale_XYZ} ${scale_XYZ} ${scale_XYZ}"/>
+			</geometry>
+		</collision>
+		<visual>
+			<origin xyz="0 0 0"
+					rpy="0 0 0"/>
+			<geometry>
+				<mesh filename="package://simulation/models/curiosity_path/meshes/suspension_arm_B2_L_fixed.dae" scale="${scale_XYZ} ${scale_XYZ} ${scale_XYZ}"/>
 			</geometry>
 		</visual>
@@ -219,12 +219,12 @@
 					rpy="0 0 0"/>
 			<geometry>
-				<mesh filename="/home/spaceros-user/src/spaceros_demo/install/mars_rover/share/mars_rover/meshes/suspension_steer_F_L_fixed.dae" scale="${scale_XYZ} ${scale_XYZ} ${scale_XYZ}"/>
-			</geometry>
-		</collision>
-		<visual>
-			<origin xyz="0 0 0"
-					rpy="0 0 0"/>
-			<geometry>
-				<mesh filename="/home/spaceros-user/src/spaceros_demo/install/mars_rover/share/mars_rover/meshes/suspension_steer_F_L_fixed.dae" scale="${scale_XYZ} ${scale_XYZ} ${scale_XYZ}"/>
+				<mesh filename="package://simulation/models/curiosity_path/meshes/suspension_steer_F_L_fixed.dae" scale="${scale_XYZ} ${scale_XYZ} ${scale_XYZ}"/>
+			</geometry>
+		</collision>
+		<visual>
+			<origin xyz="0 0 0"
+					rpy="0 0 0"/>
+			<geometry>
+				<mesh filename="package://simulation/models/curiosity_path/meshes/suspension_steer_F_L_fixed.dae" scale="${scale_XYZ} ${scale_XYZ} ${scale_XYZ}"/>
 			</geometry>
 		</visual>
@@ -346,12 +346,12 @@
 					rpy="0 0 0"/>
 			<geometry>
-				<mesh filename="/home/spaceros-user/src/spaceros_demo/install/mars_rover/share/mars_rover/meshes/suspension_steer_B_L_fixed.dae" scale="${scale_XYZ} ${scale_XYZ} ${scale_XYZ}"/>
-			</geometry>
-		</collision>
-		<visual>
-			<origin xyz="0 0 0"
-					rpy="0 0 0"/>
-			<geometry>
-				<mesh filename="/home/spaceros-user/src/spaceros_demo/install/mars_rover/share/mars_rover/meshes/suspension_steer_B_L_fixed.dae" scale="${scale_XYZ} ${scale_XYZ} ${scale_XYZ}"/>
+				<mesh filename="package://simulation/models/curiosity_path/meshes/suspension_steer_B_L_fixed.dae" scale="${scale_XYZ} ${scale_XYZ} ${scale_XYZ}"/>
+			</geometry>
+		</collision>
+		<visual>
+			<origin xyz="0 0 0"
+					rpy="0 0 0"/>
+			<geometry>
+				<mesh filename="package://simulation/models/curiosity_path/meshes/suspension_steer_B_L_fixed.dae" scale="${scale_XYZ} ${scale_XYZ} ${scale_XYZ}"/>
 			</geometry>
 		</visual>
