Commit message: paths in xacro files
Signed-off-by: Dharini Dutia <dharini@openrobotics.org>

File: models/curiosity_path/urdf/right_wheel_group.xacro (robot description, xacro)
@@ -7,12 +7,12 @@
 					rpy="0 0 0"/>
 			<geometry>
-				<mesh filename="/home/spaceros-user/src/spaceros_demo/install/mars_rover/share/mars_rover/meshes/right_axis_jointfix_v2.dae" scale="${scale_XYZ} ${scale_XYZ} ${scale_XYZ}"/>
-			</geometry>
-		</collision>
-		<visual>
-			<origin xyz="0 0 0"
-					rpy="0 0 0"/>
-			<geometry>
-				<mesh filename="/home/spaceros-user/src/spaceros_demo/install/mars_rover/share/mars_rover/meshes/right_axis_jointfix_v2.dae" scale="${scale_XYZ} ${scale_XYZ} ${scale_XYZ}"/>
+				<mesh filename="package://simulation/models/curiosity_path/meshes/right_axis_jointfix_v2.dae" scale="${scale_XYZ} ${scale_XYZ} ${scale_XYZ}"/>
+			</geometry>
+		</collision>
+		<visual>
+			<origin xyz="0 0 0"
+					rpy="0 0 0"/>
+			<geometry>
+				<mesh filename="package://simulation/models/curiosity_path/meshes/right_axis_jointfix_v2.dae" scale="${scale_XYZ} ${scale_XYZ} ${scale_XYZ}"/>
 			</geometry>
 		</visual>
@@ -38,12 +38,12 @@
 					rpy="0 0 0"/>
 			<geometry>
-				<mesh filename="/home/spaceros-user/src/spaceros_demo/install/mars_rover/share/mars_rover/meshes/suspension_arm_F_R_fixed.dae" scale="${scale_XYZ} ${scale_XYZ} ${scale_XYZ}"/>
-			</geometry>
-		</collision>
-		<visual>
-			<origin xyz="0 0 0"
-					rpy="0 0 0"/>
-			<geometry>
-				<mesh filename="/home/spaceros-user/src/spaceros_demo/install/mars_rover/share/mars_rover/meshes/suspension_arm_F_R_fixed.dae" scale="${scale_XYZ} ${scale_XYZ} ${scale_XYZ}"/>
+				<mesh filename="package://simulation/models/curiosity_path/meshes/suspension_arm_F_R_fixed.dae" scale="${scale_XYZ} ${scale_XYZ} ${scale_XYZ}"/>
+			</geometry>
+		</collision>
+		<visual>
+			<origin xyz="0 0 0"
+					rpy="0 0 0"/>
+			<geometry>
+				<mesh filename="package://simulation/models/curiosity_path/meshes/suspension_arm_F_R_fixed.dae" scale="${scale_XYZ} ${scale_XYZ} ${scale_XYZ}"/>
 			</geometry>
 		</visual>
@@ -82,12 +82,12 @@
 					rpy="0 0 0"/>
 			<geometry>
-				<mesh filename="/home/spaceros-user/src/spaceros_demo/install/mars_rover/share/mars_rover/meshes/suspension_arm_B_R_fixed.dae" scale="${scale_XYZ} ${scale_XYZ} ${scale_XYZ}"/>
-			</geometry>
-		</collision>
-		<visual>
-			<origin xyz="0 0 0"
-					rpy="0 0 0"/>
-			<geometry>
-				<mesh filename="/home/spaceros-user/src/spaceros_demo/install/mars_rover/share/mars_rover/meshes/suspension_arm_B_R_fixed.dae" scale="${scale_XYZ} ${scale_XYZ} ${scale_XYZ}"/>
+				<mesh filename="package://simulation/models/curiosity_path/meshes/suspension_arm_B_R_fixed.dae" scale="${scale_XYZ} ${scale_XYZ} ${scale_XYZ}"/>
+			</geometry>
+		</collision>
+		<visual>
+			<origin xyz="0 0 0"
+					rpy="0 0 0"/>
+			<geometry>
+				<mesh filename="package://simulation/models/curiosity_path/meshes/suspension_arm_B_R_fixed.dae" scale="${scale_XYZ} ${scale_XYZ} ${scale_XYZ}"/>
 			</geometry>
 		</visual>
@@ -150,12 +150,12 @@
 					rpy="0 0 0"/>
 			<geometry>
-				<mesh filename="/home/spaceros-user/src/spaceros_demo/install/mars_rover/share/mars_rover/meshes/suspension_arm_B2_R_fixed.dae" scale="${scale_XYZ} ${scale_XYZ} ${scale_XYZ}"/>
-			</geometry>
-		</collision>
-		<visual>
-			<origin xyz="0 0 0"
-					rpy="0 0 0"/>
-			<geometry>
-				<mesh filename="/home/spaceros-user/src/spaceros_demo/install/mars_rover/share/mars_rover/meshes/suspension_arm_B2_R_fixed.dae" scale="${scale_XYZ} ${scale_XYZ} ${scale_XYZ}"/>
+				<mesh filename="package://simulation/models/curiosity_path/meshes/suspension_arm_B2_R_fixed.dae" scale="${scale_XYZ} ${scale_XYZ} ${scale_XYZ}"/>
+			</geometry>
+		</collision>
+		<visual>
+			<origin xyz="0 0 0"
+					rpy="0 0 0"/>
+			<geometry>
+				<mesh filename="package://simulation/models/curiosity_path/meshes/suspension_arm_B2_R_fixed.dae" scale="${scale_XYZ} ${scale_XYZ} ${scale_XYZ}"/>
 			</geometry>
 		</visual>
@@ -219,12 +219,12 @@
 					rpy="0 0 0"/>
 			<geometry>
-				<mesh filename="/home/spaceros-user/src/spaceros_demo/install/mars_rover/share/mars_rover/meshes/suspension_steer_F_R_fixed.dae" scale="${scale_XYZ} ${scale_XYZ} ${scale_XYZ}"/>
-			</geometry>
-		</collision>
-		<visual>
-			<origin xyz="0 0 0"
-					rpy="0 0 0"/>
-			<geometry>
-				<mesh filename="/home/spaceros-user/src/spaceros_demo/install/mars_rover/share/mars_rover/meshes/suspension_steer_F_R_fixed.dae" scale="${scale_XYZ} ${scale_XYZ} ${scale_XYZ}"/>
+				<mesh filename="package://simulation/models/curiosity_path/meshes/suspension_steer_F_R_fixed.dae" scale="${scale_XYZ} ${scale_XYZ} ${scale_XYZ}"/>
+			</geometry>
+		</collision>
+		<visual>
+			<origin xyz="0 0 0"
+					rpy="0 0 0"/>
+			<geometry>
+				<mesh filename="package://simulation/models/curiosity_path/meshes/suspension_steer_F_R_fixed.dae" scale="${scale_XYZ} ${scale_XYZ} ${scale_XYZ}"/>
 			</geometry>
 		</visual>
@@ -344,12 +344,12 @@
 					rpy="0 0 0"/>
 			<geometry>
-				<mesh filename="/home/spaceros-user/src/spaceros_demo/install/mars_rover/share/mars_rover/meshes/suspension_steer_B_R_fixed.dae" scale="${scale_XYZ} ${scale_XYZ} ${scale_XYZ}"/>
-			</geometry>
-		</collision>
-		<visual>
-			<origin xyz="0 0 0"
-					rpy="0 0 0"/>
-			<geometry>
-				<mesh filename="/home/spaceros-user/src/spaceros_demo/install/mars_rover/share/mars_rover/meshes/suspension_steer_B_R_fixed.dae" scale="${scale_XYZ} ${scale_XYZ} ${scale_XYZ}"/>
+				<mesh filename="package://simulation/models/curiosity_path/meshes/suspension_steer_B_R_fixed.dae" scale="${scale_XYZ} ${scale_XYZ} ${scale_XYZ}"/>
+			</geometry>
+		</collision>
+		<visual>
+			<origin xyz="0 0 0"
+					rpy="0 0 0"/>
+			<geometry>
+				<mesh filename="package://simulation/models/curiosity_path/meshes/suspension_steer_B_R_fixed.dae" scale="${scale_XYZ} ${scale_XYZ} ${scale_XYZ}"/>
 			</geometry>
 		</visual>

File: models/curiosity_path/urdf/sensor_mast.xacro (robot description, xacro)
@@ -31,5 +31,5 @@
 					rpy="0 0 0"/>
 			<geometry>
-				<mesh filename="/home/spaceros-user/src/spaceros_demo/install/mars_rover/share/mars_rover/meshes/mast_p_fixed.dae" scale="${scale_XYZ} ${scale_XYZ} ${scale_XYZ}"/>
+				<mesh filename="package://simulation/models/curiosity_path/meshes/mast_p_fixed.dae" scale="${scale_XYZ} ${scale_XYZ} ${scale_XYZ}"/>
 			</geometry>
 		</collision>
@@ -38,5 +38,5 @@
 					rpy="0 0 0"/>
 			<geometry>
-				<mesh filename="/home/spaceros-user/src/spaceros_demo/install/mars_rover/share/mars_rover/meshes/mast_p_fixed.dae" scale="${scale_XYZ} ${scale_XYZ} ${scale_XYZ}"/>
+				<mesh filename="package://simulation/models/curiosity_path/meshes/mast_p_fixed.dae" scale="${scale_XYZ} ${scale_XYZ} ${scale_XYZ}"/>
 			</geometry>
 		</visual>
@@ -99,5 +99,5 @@
 					rpy="0 0 0"/>
 			<geometry>
-				<mesh filename="/home/spaceros-user/src/spaceros_demo/install/mars_rover/share/mars_rover/meshes/mast_02_fixed.dae" scale="${scale_XYZ} ${scale_XYZ} ${scale_XYZ}"/>
+				<mesh filename="package://simulation/models/curiosity_path/meshes/mast_02_fixed.dae" scale="${scale_XYZ} ${scale_XYZ} ${scale_XYZ}"/>
 			</geometry>
 		</collision>
@@ -106,5 +106,5 @@
 					rpy="0 0 0"/>
 			<geometry>
-				<mesh filename="/home/spaceros-user/src/spaceros_demo/install/mars_rover/share/mars_rover/meshes/mast_02_fixed.dae" scale="${scale_XYZ} ${scale_XYZ} ${scale_XYZ}"/>
+				<mesh filename="package://simulation/models/curiosity_path/meshes/mast_02_fixed.dae" scale="${scale_XYZ} ${scale_XYZ} ${scale_XYZ}"/>
 			</geometry>
 		</visual>
@@ -167,5 +167,5 @@
 					rpy="0 0 0"/>
 			<geometry>
-				<mesh filename="/home/spaceros-user/src/spaceros_demo/install/mars_rover/share/mars_rover/meshes/mast_cameras.dae" scale="${scale_XYZ} ${scale_XYZ} ${scale_XYZ}"/>
+				<mesh filename="package://simulation/models/curiosity_path/meshes/mast_cameras.dae" scale="${scale_XYZ} ${scale_XYZ} ${scale_XYZ}"/>
 			</geometry>
 		</collision>
@@ -174,5 +174,5 @@
 					rpy="0 0 0"/>
 			<geometry>
-				<mesh filename="/home/spaceros-user/src/spaceros_demo/install/mars_rover/share/mars_rover/meshes/mast_cameras.dae" scale="${scale_XYZ} ${scale_XYZ} ${scale_XYZ}"/>
+				<mesh filename="package://simulation/models/curiosity_path/meshes/mast_cameras.dae" scale="${scale_XYZ} ${scale_XYZ} ${scale_XYZ}"/>
 			</geometry>
 		</visual>

File: models/curiosity_path/urdf/wheel.xacro (robot description, xacro)
@@ -15,5 +15,5 @@
 					rpy="0 0 0"/>
 			<geometry>
-				<mesh filename="/home/spaceros-user/src/spaceros_demo/install/mars_rover/share/mars_rover/meshes/wheel_fixed.dae" scale="${scale_XYZ} ${scale_XYZ} ${scale_XYZ}"/>
+				<mesh filename="package://simulation/models/curiosity_path/meshes/wheel_fixed.dae" scale="${scale_XYZ} ${scale_XYZ} ${scale_XYZ}"/>
 			</geometry>
 		</visual>
