Commit message: Use file:\\ prefix for mesh filenames

File: models/curiosity_path/urdf/arm.xacro (robot description, xacro)
@@ -31,12 +31,12 @@
 					rpy="0 0 0"/>
 			<geometry>
-				<mesh filename="$(find simulation)/models/curiosity_path/meshes/arm_01_fixed.dae" scale="${scale_XYZ} ${scale_XYZ} ${scale_XYZ}"/>
-			</geometry>
-		</collision>
-		<visual>
-			<origin xyz="0 0 0"
-					rpy="0 0 0"/>
-			<geometry>
-				<mesh filename="$(find simulation)/models/curiosity_path/meshes/arm_01_fixed.dae" scale="${scale_XYZ} ${scale_XYZ} ${scale_XYZ}"/>
+				<mesh filename="file:///$(find simulation)/models/curiosity_path/meshes/arm_01_fixed.dae" scale="${scale_XYZ} ${scale_XYZ} ${scale_XYZ}"/>
+			</geometry>
+		</collision>
+		<visual>
+			<origin xyz="0 0 0"
+					rpy="0 0 0"/>
+			<geometry>
+				<mesh filename="file:///$(find simulation)/models/curiosity_path/meshes/arm_01_fixed.dae" scale="${scale_XYZ} ${scale_XYZ} ${scale_XYZ}"/>
 			</geometry>
 		</visual>
@@ -99,12 +99,12 @@
 					rpy="0 0 0"/>
 			<geometry>
-				<mesh filename="$(find simulation)/models/curiosity_path/meshes/arm_01_fixed.dae" scale="${scale_XYZ} ${scale_XYZ} ${scale_XYZ}"/>
-			</geometry>
-		</collision>
-		<visual>
-			<origin xyz="0 0 0"
-					rpy="0 0 0"/>
-			<geometry>
-				<mesh filename="$(find simulation)/models/curiosity_path/meshes/arm_02_fixed.dae" scale="${scale_XYZ} ${scale_XYZ} ${scale_XYZ}"/>
+				<mesh filename="file:///$(find simulation)/models/curiosity_path/meshes/arm_01_fixed.dae" scale="${scale_XYZ} ${scale_XYZ} ${scale_XYZ}"/>
+			</geometry>
+		</collision>
+		<visual>
+			<origin xyz="0 0 0"
+					rpy="0 0 0"/>
+			<geometry>
+				<mesh filename="file:///$(find simulation)/models/curiosity_path/meshes/arm_02_fixed.dae" scale="${scale_XYZ} ${scale_XYZ} ${scale_XYZ}"/>
 			</geometry>
 		</visual>
@@ -167,12 +167,12 @@
 					rpy="0 0 0"/>
 			<geometry>
-				<mesh filename="$(find simulation)/models/curiosity_path/meshes/arm_03_fixed.dae" scale="${scale_XYZ} ${scale_XYZ} ${scale_XYZ}"/>
-			</geometry>
-		</collision>
-		<visual>
-			<origin xyz="0 0 0"
-					rpy="0 0 0"/>
-			<geometry>
-				<mesh filename="$(find simulation)/models/curiosity_path/meshes/arm_03_fixed.dae" scale="${scale_XYZ} ${scale_XYZ} ${scale_XYZ}"/>
+				<mesh filename="file:///$(find simulation)/models/curiosity_path/meshes/arm_03_fixed.dae" scale="${scale_XYZ} ${scale_XYZ} ${scale_XYZ}"/>
+			</geometry>
+		</collision>
+		<visual>
+			<origin xyz="0 0 0"
+					rpy="0 0 0"/>
+			<geometry>
+				<mesh filename="file:///$(find simulation)/models/curiosity_path/meshes/arm_03_fixed.dae" scale="${scale_XYZ} ${scale_XYZ} ${scale_XYZ}"/>
 			</geometry>
 		</visual>
@@ -235,12 +235,12 @@
 					rpy="0 0 0"/>
 			<geometry>
-				<mesh filename="$(find simulation)/models/curiosity_path/meshes/arm_04_fixed.dae" scale="${scale_XYZ} ${scale_XYZ} ${scale_XYZ}"/>
-			</geometry>
-		</collision>
-		<visual>
-			<origin xyz="0 0 0"
-					rpy="0 0 0"/>
-			<geometry>
-				<mesh filename="$(find simulation)/models/curiosity_path/meshes/arm_04_fixed.dae" scale="${scale_XYZ} ${scale_XYZ} ${scale_XYZ}"/>
+				<mesh filename="file:///$(find simulation)/models/curiosity_path/meshes/arm_04_fixed.dae" scale="${scale_XYZ} ${scale_XYZ} ${scale_XYZ}"/>
+			</geometry>
+		</collision>
+		<visual>
+			<origin xyz="0 0 0"
+					rpy="0 0 0"/>
+			<geometry>
+				<mesh filename="file:///$(find simulation)/models/curiosity_path/meshes/arm_04_fixed.dae" scale="${scale_XYZ} ${scale_XYZ} ${scale_XYZ}"/>
 			</geometry>
 		</visual>
@@ -303,12 +303,12 @@
 					rpy="0 0 0"/>
 			<geometry>
-				<mesh filename="$(find simulation)/models/curiosity_path/meshes/arm_tools_fixed.dae" scale="${scale_XYZ} ${scale_XYZ} ${scale_XYZ}"/>
-			</geometry>
-		</collision>
-		<visual>
-			<origin xyz="0 0 0"
-					rpy="0 0 0"/>
-			<geometry>
-				<mesh filename="$(find simulation)/models/curiosity_path/meshes/arm_tools_fixed.dae" scale="${scale_XYZ} ${scale_XYZ} ${scale_XYZ}"/>
+				<mesh filename="file:///$(find simulation)/models/curiosity_path/meshes/arm_tools_fixed.dae" scale="${scale_XYZ} ${scale_XYZ} ${scale_XYZ}"/>
+			</geometry>
+		</collision>
+		<visual>
+			<origin xyz="0 0 0"
+					rpy="0 0 0"/>
+			<geometry>
+				<mesh filename="file:///$(find simulation)/models/curiosity_path/meshes/arm_tools_fixed.dae" scale="${scale_XYZ} ${scale_XYZ} ${scale_XYZ}"/>
 			</geometry>
 		</visual>

File: models/curiosity_path/urdf/chassis.xacro (robot description, xacro)
@@ -19,5 +19,5 @@
 					rpy="0 0 0"/>
 			<geometry>
-				<mesh filename="$(find simulation)/models/curiosity_path/meshes/chassis_full_fixed_glitch_v2.dae" scale="${scale_XYZ} ${scale_XYZ} ${scale_XYZ}"/>
+				<mesh filename="file:///$(find simulation)/models/curiosity_path/meshes/chassis_full_fixed_glitch_v2.dae" scale="${scale_XYZ} ${scale_XYZ} ${scale_XYZ}"/>
 			</geometry>
 		</collision>
@@ -26,5 +26,5 @@
 					rpy="0 0 0"/>
 			<geometry>
-				<mesh filename="$(find simulation)/models/curiosity_path/meshes/chassis_full_fixed_glitch_v2.dae" scale="${scale_XYZ} ${scale_XYZ} ${scale_XYZ}"/>
+				<mesh filename="file:///$(find simulation)/models/curiosity_path/meshes/chassis_full_fixed_glitch_v2.dae" scale="${scale_XYZ} ${scale_XYZ} ${scale_XYZ}"/>
 			</geometry>
 		</visual>

File: models/curiosity_path/urdf/left_wheel_group.xacro (robot description, xacro)
@@ -7,12 +7,12 @@
 					rpy="0 0 0"/>
 			<geometry>
-				<mesh filename="$(find simulation)/models/curiosity_path/meshes/left_axis_jointfix_v2.dae" scale="${scale_XYZ} ${scale_XYZ} ${scale_XYZ}"/>
-			</geometry>
-		</collision>
-		<visual>
-			<origin xyz="0 0 0"
-					rpy="0 0 0"/>
-			<geometry>
-				<mesh filename="$(find simulation)/models/curiosity_path/meshes/left_axis_jointfix_v2.dae" scale="${scale_XYZ} ${scale_XYZ} ${scale_XYZ}"/>
+				<mesh filename="file:///$(find simulation)/models/curiosity_path/meshes/left_axis_jointfix_v2.dae" scale="${scale_XYZ} ${scale_XYZ} ${scale_XYZ}"/>
+			</geometry>
+		</collision>
+		<visual>
+			<origin xyz="0 0 0"
+					rpy="0 0 0"/>
+			<geometry>
+				<mesh filename="file:///$(find simulation)/models/curiosity_path/meshes/left_axis_jointfix_v2.dae" scale="${scale_XYZ} ${scale_XYZ} ${scale_XYZ}"/>
 			</geometry>
 		</visual>
@@ -38,12 +38,12 @@
 					rpy="0 0 0"/>
 			<geometry>
-				<mesh filename="$(find simulation)/models/curiosity_path/meshes/suspension_arm_F_L_fixed.dae" scale="${scale_XYZ} ${scale_XYZ} ${scale_XYZ}"/>
-			</geometry>
-		</collision>
-		<visual>
-			<origin xyz="0 0 0"
-					rpy="0 0 0"/>
-			<geometry>
-				<mesh filename="$(find simulation)/models/curiosity_path/meshes/suspension_arm_F_L_fixed.dae" scale="${scale_XYZ} ${scale_XYZ} ${scale_XYZ}"/>
+				<mesh filename="file:///$(find simulation)/models/curiosity_path/meshes/suspension_arm_F_L_fixed.dae" scale="${scale_XYZ} ${scale_XYZ} ${scale_XYZ}"/>
+			</geometry>
+		</collision>
+		<visual>
+			<origin xyz="0 0 0"
+					rpy="0 0 0"/>
+			<geometry>
+				<mesh filename="file:///$(find simulation)/models/curiosity_path/meshes/suspension_arm_F_L_fixed.dae" scale="${scale_XYZ} ${scale_XYZ} ${scale_XYZ}"/>
 			</geometry>
 		</visual>
@@ -82,12 +82,12 @@
 					rpy="0 0 0"/>
 			<geometry>
-				<mesh filename="$(find simulation)/models/curiosity_path/meshes/suspension_arm_B_L_fixed.dae" scale="${scale_XYZ} ${scale_XYZ} ${scale_XYZ}"/>
-			</geometry>
-		</collision>
-		<visual>
-			<origin xyz="0 0 0"
-					rpy="0 0 0"/>
-			<geometry>
-				<mesh filename="$(find simulation)/models/curiosity_path/meshes/suspension_arm_B_L_fixed.dae" scale="${scale_XYZ} ${scale_XYZ} ${scale_XYZ}"/>
+				<mesh filename="file:///$(find simulation)/models/curiosity_path/meshes/suspension_arm_B_L_fixed.dae" scale="${scale_XYZ} ${scale_XYZ} ${scale_XYZ}"/>
+			</geometry>
+		</collision>
+		<visual>
+			<origin xyz="0 0 0"
+					rpy="0 0 0"/>
+			<geometry>
+				<mesh filename="file:///$(find simulation)/models/curiosity_path/meshes/suspension_arm_B_L_fixed.dae" scale="${scale_XYZ} ${scale_XYZ} ${scale_XYZ}"/>
 			</geometry>
 		</visual>
@@ -150,12 +150,12 @@
 					rpy="0 0 0"/>
 			<geometry>
-				<mesh filename="$(find simulation)/models/curiosity_path/meshes/suspension_arm_B2_L_fixed.dae" scale="${scale_XYZ} ${scale_XYZ} ${scale_XYZ}"/>
-			</geometry>
-		</collision>
-		<visual>
-			<origin xyz="0 0 0"
-					rpy="0 0 0"/>
-			<geometry>
-				<mesh filename="$(find simulation)/models/curiosity_path/meshes/suspension_arm_B2_L_fixed.dae" scale="${scale_XYZ} ${scale_XYZ} ${scale_XYZ}"/>
+				<mesh filename="file:///$(find simulation)/models/curiosity_path/meshes/suspension_arm_B2_L_fixed.dae" scale="${scale_XYZ} ${scale_XYZ} ${scale_XYZ}"/>
+			</geometry>
+		</collision>
+		<visual>
+			<origin xyz="0 0 0"
+					rpy="0 0 0"/>
+			<geometry>
+				<mesh filename="file:///$(find simulation)/models/curiosity_path/meshes/suspension_arm_B2_L_fixed.dae" scale="${scale_XYZ} ${scale_XYZ} ${scale_XYZ}"/>
 			</geometry>
 		</visual>
@@ -219,12 +219,12 @@
 					rpy="0 0 0"/>
 			<geometry>
-				<mesh filename="$(find simulation)/models/curiosity_path/meshes/suspension_steer_F_L_fixed.dae" scale="${scale_XYZ} ${scale_XYZ} ${scale_XYZ}"/>
-			</geometry>
-		</collision>
-		<visual>
-			<origin xyz="0 0 0"
-					rpy="0 0 0"/>
-			<geometry>
-				<mesh filename="$(find simulation)/models/curiosity_path/meshes/suspension_steer_F_L_fixed.dae" scale="${scale_XYZ} ${scale_XYZ} ${scale_XYZ}"/>
+				<mesh filename="file:///$(find simulation)/models/curiosity_path/meshes/suspension_steer_F_L_fixed.dae" scale="${scale_XYZ} ${scale_XYZ} ${scale_XYZ}"/>
+			</geometry>
+		</collision>
+		<visual>
+			<origin xyz="0 0 0"
+					rpy="0 0 0"/>
+			<geometry>
+				<mesh filename="file:///$(find simulation)/models/curiosity_path/meshes/suspension_steer_F_L_fixed.dae" scale="${scale_XYZ} ${scale_XYZ} ${scale_XYZ}"/>
 			</geometry>
 		</visual>
@@ -346,12 +346,12 @@
 					rpy="0 0 0"/>
 			<geometry>
-				<mesh filename="$(find simulation)/models/curiosity_path/meshes/suspension_steer_B_L_fixed.dae" scale="${scale_XYZ} ${scale_XYZ} ${scale_XYZ}"/>
-			</geometry>
-		</collision>
-		<visual>
-			<origin xyz="0 0 0"
-					rpy="0 0 0"/>
-			<geometry>
-				<mesh filename="$(find simulation)/models/curiosity_path/meshes/suspension_steer_B_L_fixed.dae" scale="${scale_XYZ} ${scale_XYZ} ${scale_XYZ}"/>
+				<mesh filename="file:///$(find simulation)/models/curiosity_path/meshes/suspension_steer_B_L_fixed.dae" scale="${scale_XYZ} ${scale_XYZ} ${scale_XYZ}"/>
+			</geometry>
+		</collision>
+		<visual>
+			<origin xyz="0 0 0"
+					rpy="0 0 0"/>
+			<geometry>
+				<mesh filename="file:///$(find simulation)/models/curiosity_path/meshes/suspension_steer_B_L_fixed.dae" scale="${scale_XYZ} ${scale_XYZ} ${scale_XYZ}"/>
 			</geometry>
 		</visual>

File: models/curiosity_path/urdf/right_wheel_group.xacro (robot description, xacro)
@@ -7,12 +7,12 @@
 					rpy="0 0 0"/>
 			<geometry>
-				<mesh filename="$(find simulation)/models/curiosity_path/meshes/right_axis_jointfix_v2.dae" scale="${scale_XYZ} ${scale_XYZ} ${scale_XYZ}"/>
-			</geometry>
-		</collision>
-		<visual>
-			<origin xyz="0 0 0"
-					rpy="0 0 0"/>
-			<geometry>
-				<mesh filename="$(find simulation)/models/curiosity_path/meshes/right_axis_jointfix_v2.dae" scale="${scale_XYZ} ${scale_XYZ} ${scale_XYZ}"/>
+				<mesh filename="file:///$(find simulation)/models/curiosity_path/meshes/right_axis_jointfix_v2.dae" scale="${scale_XYZ} ${scale_XYZ} ${scale_XYZ}"/>
+			</geometry>
+		</collision>
+		<visual>
+			<origin xyz="0 0 0"
+					rpy="0 0 0"/>
+			<geometry>
+				<mesh filename="file:///$(find simulation)/models/curiosity_path/meshes/right_axis_jointfix_v2.dae" scale="${scale_XYZ} ${scale_XYZ} ${scale_XYZ}"/>
 			</geometry>
 		</visual>
@@ -38,12 +38,12 @@
 					rpy="0 0 0"/>
 			<geometry>
-				<mesh filename="$(find simulation)/models/curiosity_path/meshes/suspension_arm_F_R_fixed.dae" scale="${scale_XYZ} ${scale_XYZ} ${scale_XYZ}"/>
-			</geometry>
-		</collision>
-		<visual>
-			<origin xyz="0 0 0"
-					rpy="0 0 0"/>
-			<geometry>
-				<mesh filename="$(find simulation)/models/curiosity_path/meshes/suspension_arm_F_R_fixed.dae" scale="${scale_XYZ} ${scale_XYZ} ${scale_XYZ}"/>
+				<mesh filename="file:///$(find simulation)/models/curiosity_path/meshes/suspension_arm_F_R_fixed.dae" scale="${scale_XYZ} ${scale_XYZ} ${scale_XYZ}"/>
+			</geometry>
+		</collision>
+		<visual>
+			<origin xyz="0 0 0"
+					rpy="0 0 0"/>
+			<geometry>
+				<mesh filename="file:///$(find simulation)/models/curiosity_path/meshes/suspension_arm_F_R_fixed.dae" scale="${scale_XYZ} ${scale_XYZ} ${scale_XYZ}"/>
 			</geometry>
 		</visual>
@@ -82,12 +82,12 @@
 					rpy="0 0 0"/>
 			<geometry>
-				<mesh filename="$(find simulation)/models/curiosity_path/meshes/suspension_arm_B_R_fixed.dae" scale="${scale_XYZ} ${scale_XYZ} ${scale_XYZ}"/>
-			</geometry>
-		</collision>
-		<visual>
-			<origin xyz="0 0 0"
-					rpy="0 0 0"/>
-			<geometry>
-				<mesh filename="$(find simulation)/models/curiosity_path/meshes/suspension_arm_B_R_fixed.dae" scale="${scale_XYZ} ${scale_XYZ} ${scale_XYZ}"/>
+				<mesh filename="file:///$(find simulation)/models/curiosity_path/meshes/suspension_arm_B_R_fixed.dae" scale="${scale_XYZ} ${scale_XYZ} ${scale_XYZ}"/>
+			</geometry>
+		</collision>
+		<visual>
+			<origin xyz="0 0 0"
+					rpy="0 0 0"/>
+			<geometry>
+				<mesh filename="file:///$(find simulation)/models/curiosity_path/meshes/suspension_arm_B_R_fixed.dae" scale="${scale_XYZ} ${scale_XYZ} ${scale_XYZ}"/>
 			</geometry>
 		</visual>
@@ -150,12 +150,12 @@
 					rpy="0 0 0"/>
 			<geometry>
-				<mesh filename="$(find simulation)/models/curiosity_path/meshes/suspension_arm_B2_R_fixed.dae" scale="${scale_XYZ} ${scale_XYZ} ${scale_XYZ}"/>
-			</geometry>
-		</collision>
-		<visual>
-			<origin xyz="0 0 0"
-					rpy="0 0 0"/>
-			<geometry>
-				<mesh filename="$(find simulation)/models/curiosity_path/meshes/suspension_arm_B2_R_fixed.dae" scale="${scale_XYZ} ${scale_XYZ} ${scale_XYZ}"/>
+				<mesh filename="file:///$(find simulation)/models/curiosity_path/meshes/suspension_arm_B2_R_fixed.dae" scale="${scale_XYZ} ${scale_XYZ} ${scale_XYZ}"/>
+			</geometry>
+		</collision>
+		<visual>
+			<origin xyz="0 0 0"
+					rpy="0 0 0"/>
+			<geometry>
+				<mesh filename="file:///$(find simulation)/models/curiosity_path/meshes/suspension_arm_B2_R_fixed.dae" scale="${scale_XYZ} ${scale_XYZ} ${scale_XYZ}"/>
 			</geometry>
 		</visual>
@@ -219,12 +219,12 @@
 					rpy="0 0 0"/>
 			<geometry>
-				<mesh filename="$(find simulation)/models/curiosity_path/meshes/suspension_steer_F_R_fixed.dae" scale="${scale_XYZ} ${scale_XYZ} ${scale_XYZ}"/>
-			</geometry>
-		</collision>
-		<visual>
-			<origin xyz="0 0 0"
-					rpy="0 0 0"/>
-			<geometry>
-				<mesh filename="$(find simulation)/models/curiosity_path/meshes/suspension_steer_F_R_fixed.dae" scale="${scale_XYZ} ${scale_XYZ} ${scale_XYZ}"/>
+				<mesh filename="file:///$(find simulation)/models/curiosity_path/meshes/suspension_steer_F_R_fixed.dae" scale="${scale_XYZ} ${scale_XYZ} ${scale_XYZ}"/>
+			</geometry>
+		</collision>
+		<visual>
+			<origin xyz="0 0 0"
+					rpy="0 0 0"/>
+			<geometry>
+				<mesh filename="file:///$(find simulation)/models/curiosity_path/meshes/suspension_steer_F_R_fixed.dae" scale="${scale_XYZ} ${scale_XYZ} ${scale_XYZ}"/>
 			</geometry>
 		</visual>
@@ -344,12 +344,12 @@
 					rpy="0 0 0"/>
 			<geometry>
-				<mesh filename="$(find simulation)/models/curiosity_path/meshes/suspension_steer_B_R_fixed.dae" scale="${scale_XYZ} ${scale_XYZ} ${scale_XYZ}"/>
-			</geometry>
-		</collision>
-		<visual>
-			<origin xyz="0 0 0"
-					rpy="0 0 0"/>
-			<geometry>
-				<mesh filename="$(find simulation)/models/curiosity_path/meshes/suspension_steer_B_R_fixed.dae" scale="${scale_XYZ} ${scale_XYZ} ${scale_XYZ}"/>
+				<mesh filename="file:///$(find simulation)/models/curiosity_path/meshes/suspension_steer_B_R_fixed.dae" scale="${scale_XYZ} ${scale_XYZ} ${scale_XYZ}"/>
+			</geometry>
+		</collision>
+		<visual>
+			<origin xyz="0 0 0"
+					rpy="0 0 0"/>
+			<geometry>
+				<mesh filename="file:///$(find simulation)/models/curiosity_path/meshes/suspension_steer_B_R_fixed.dae" scale="${scale_XYZ} ${scale_XYZ} ${scale_XYZ}"/>
 			</geometry>
 		</visual>

File: models/curiosity_path/urdf/sensor_mast.xacro (robot description, xacro)
@@ -31,5 +31,5 @@
 					rpy="0 0 0"/>
 			<geometry>
-				<mesh filename="$(find simulation)/models/curiosity_path/meshes/mast_p_fixed.dae" scale="${scale_XYZ} ${scale_XYZ} ${scale_XYZ}"/>
+				<mesh filename="file:///$(find simulation)/models/curiosity_path/meshes/mast_p_fixed.dae" scale="${scale_XYZ} ${scale_XYZ} ${scale_XYZ}"/>
 			</geometry>
 		</collision>
@@ -38,5 +38,5 @@
 					rpy="0 0 0"/>
 			<geometry>
-				<mesh filename="$(find simulation)/models/curiosity_path/meshes/mast_p_fixed.dae" scale="${scale_XYZ} ${scale_XYZ} ${scale_XYZ}"/>
+				<mesh filename="file:///$(find simulation)/models/curiosity_path/meshes/mast_p_fixed.dae" scale="${scale_XYZ} ${scale_XYZ} ${scale_XYZ}"/>
 			</geometry>
 		</visual>
@@ -99,5 +99,5 @@
 					rpy="0 0 0"/>
 			<geometry>
-				<mesh filename="$(find simulation)/models/curiosity_path/meshes/mast_02_fixed.dae" scale="${scale_XYZ} ${scale_XYZ} ${scale_XYZ}"/>
+				<mesh filename="file:///$(find simulation)/models/curiosity_path/meshes/mast_02_fixed.dae" scale="${scale_XYZ} ${scale_XYZ} ${scale_XYZ}"/>
 			</geometry>
 		</collision>
@@ -106,5 +106,5 @@
 					rpy="0 0 0"/>
 			<geometry>
-				<mesh filename="$(find simulation)/models/curiosity_path/meshes/mast_02_fixed.dae" scale="${scale_XYZ} ${scale_XYZ} ${scale_XYZ}"/>
+				<mesh filename="file:///$(find simulation)/models/curiosity_path/meshes/mast_02_fixed.dae" scale="${scale_XYZ} ${scale_XYZ} ${scale_XYZ}"/>
 			</geometry>
 		</visual>
@@ -167,5 +167,5 @@
 					rpy="0 0 0"/>
 			<geometry>
-				<mesh filename="$(find simulation)/models/curiosity_path/meshes/mast_cameras.dae" scale="${scale_XYZ} ${scale_XYZ} ${scale_XYZ}"/>
+				<mesh filename="file:///$(find simulation)/models/curiosity_path/meshes/mast_cameras.dae" scale="${scale_XYZ} ${scale_XYZ} ${scale_XYZ}"/>
 			</geometry>
 		</collision>
@@ -174,5 +174,5 @@
 					rpy="0 0 0"/>
 			<geometry>
-				<mesh filename="$(find simulation)/models/curiosity_path/meshes/mast_cameras.dae" scale="${scale_XYZ} ${scale_XYZ} ${scale_XYZ}"/>
+				<mesh filename="file:///$(find simulation)/models/curiosity_path/meshes/mast_cameras.dae" scale="${scale_XYZ} ${scale_XYZ} ${scale_XYZ}"/>
 			</geometry>
 		</visual>

File: models/curiosity_path/urdf/wheel.xacro (robot description, xacro)
@@ -15,5 +15,5 @@
 					rpy="0 0 0"/>
 			<geometry>
-				<mesh filename="$(find simulation)/models/curiosity_path/meshes/wheel_fixed.dae" scale="${scale_XYZ} ${scale_XYZ} ${scale_XYZ}"/>
+				<mesh filename="file:///$(find simulation)/models/curiosity_path/meshes/wheel_fixed.dae" scale="${scale_XYZ} ${scale_XYZ} ${scale_XYZ}"/>
 			</geometry>
 		</visual>
