Commit message: Separated the transmission data which is not currently used by ros2 control

File: models/curiosity_path/urdf/arm.xacro (robot description, xacro)
@@ -28,9 +28,8 @@
 	<link name='arm_01'>
 		<collision>
-			<origin xyz="0 0 0"
-					rpy="0 0 0"/>
-			<geometry>
-				<mesh filename="package://simulation/models/curiosity_path/meshes/arm_01_fixed.dae" scale="${scale_XYZ} ${scale_XYZ} ${scale_XYZ}"/>
-			</geometry>
+		    <origin xyz="0 0 0" rpy="0 0 0"/>
+		    <geometry>
+		        <mesh filename="package://simulation/models/curiosity_path/meshes/arm_01_fixed.dae" scale="${scale_XYZ} ${scale_XYZ} ${scale_XYZ}"/>
+		    </geometry>
 		</collision>
 		<visual>
@@ -60,14 +59,4 @@
         <dynamics damping="0.0" friction="0.0"/>
 	</joint>
-    <transmission name="arm_01_trans">
-      <type>transmission_interface/SimpleTransmission</type>
-      <joint name="arm_01_joint">
-        <hardwareInterface>hardware_interface/EffortJointInterface</hardwareInterface>
-      </joint>
-      <actuator name="arm_01Motor">
-        <hardwareInterface>hardware_interface/EffortJointInterface</hardwareInterface>
-        <mechanicalReduction>1</mechanicalReduction>
-      </actuator>
-    </transmission>
   	<link name='arm_01_to_arm_02'>
 		<inertial>
@@ -128,14 +117,4 @@
         <dynamics damping="0.0" friction="0.0"/>
 	</joint>
-    <transmission name="arm_02_trans">
-      <type>transmission_interface/SimpleTransmission</type>
-      <joint name="arm_02_joint">
-        <hardwareInterface>hardware_interface/EffortJointInterface</hardwareInterface>
-      </joint>
-      <actuator name="arm_02Motor">
-        <hardwareInterface>hardware_interface/EffortJointInterface</hardwareInterface>
-        <mechanicalReduction>1</mechanicalReduction>
-      </actuator>
-    </transmission>
   	<link name='arm_02_to_arm_03'>
 		<inertial>
@@ -196,14 +175,4 @@
         <dynamics damping="0.0" friction="0.0"/>
 	</joint>
-    <transmission name="arm_03_trans">
-      <type>transmission_interface/SimpleTransmission</type>
-      <joint name="arm_03_joint">
-        <hardwareInterface>hardware_interface/EffortJointInterface</hardwareInterface>
-      </joint>
-      <actuator name="arm_03Motor">
-        <hardwareInterface>hardware_interface/EffortJointInterface</hardwareInterface>
-        <mechanicalReduction>1</mechanicalReduction>
-      </actuator>
-    </transmission>
   	<link name='arm_03_to_arm_04'>
 		<inertial>
@@ -232,6 +201,5 @@
   	<link name='arm_04'>
 		<collision>
-			<origin xyz="0 0 0"
-					rpy="0 0 0"/>
+			<origin xyz="0 0 0" rpy="0 0 0"/>
 			<geometry>
 				<mesh filename="package://simulation/models/curiosity_path/meshes/arm_04_fixed.dae" scale="${scale_XYZ} ${scale_XYZ} ${scale_XYZ}"/>
@@ -239,6 +207,5 @@
 		</collision>
 		<visual>
-			<origin xyz="0 0 0"
-					rpy="0 0 0"/>
+			<origin xyz="0 0 0" rpy="0 0 0"/>
 			<geometry>
 				<mesh filename="package://simulation/models/curiosity_path/meshes/arm_04_fixed.dae" scale="${scale_XYZ} ${scale_XYZ} ${scale_XYZ}"/>
@@ -246,6 +213,5 @@
 		</visual>
 		<inertial>
-			<origin xyz="0 0 0"
-					rpy="0 0 0"/>
+			<origin xyz="0 0 0" rpy="0 0 0"/>
 			<mass value="${arm_04_Mass}"/>
 			<xacro:box_inertia
@@ -264,16 +230,6 @@
         <dynamics damping="0.0" friction="0.0"/>
 	</joint>
-    <transmission name="arm_04_trans">
-      <type>transmission_interface/SimpleTransmission</type>
-      <joint name="arm_04_joint">
-        <hardwareInterface>hardware_interface/EffortJointInterface</hardwareInterface>
-      </joint>
-      <actuator name="arm_04Motor">
-        <hardwareInterface>hardware_interface/EffortJointInterface</hardwareInterface>
-        <mechanicalReduction>1</mechanicalReduction>
-      </actuator>
-    </transmission>
   	<link name='arm_04_to_arm_tools'>
-		<inertial>
+	<inertial>
             <origin xyz="0 0 0" rpy="0 0 0"/>
             <mass value="0.02" />
@@ -300,6 +256,5 @@
   	<link name='arm_tools'>
 		<collision>
-			<origin xyz="0 0 0"
-					rpy="0 0 0"/>
+			<origin xyz="0 0 0" rpy="0 0 0"/>
 			<geometry>
 				<mesh filename="package://simulation/models/curiosity_path/meshes/arm_tools_fixed.dae" scale="${scale_XYZ} ${scale_XYZ} ${scale_XYZ}"/>
@@ -307,6 +262,5 @@
 		</collision>
 		<visual>
-			<origin xyz="0 0 0"
-					rpy="0 0 0"/>
+			<origin xyz="0 0 0" rpy="0 0 0"/>
 			<geometry>
 				<mesh filename="package://simulation/models/curiosity_path/meshes/arm_tools_fixed.dae" scale="${scale_XYZ} ${scale_XYZ} ${scale_XYZ}"/>
@@ -314,6 +268,5 @@
 		</visual>
 		<inertial>
-			<origin xyz="0 0 0"
-					rpy="0 0 0"/>
+			<origin xyz="0 0 0" rpy="0 0 0"/>
 			<mass value="${arm_tools_Mass}"/>
 			<xacro:box_inertia
@@ -332,11 +285,54 @@
         <dynamics damping="0.0" friction="0.0"/>
 	</joint>
+  </xacro:macro>
+  <!-- ros2_control transmission does NOT use this currently. This macro is not actively used -->
+  <xacro:macro name="arm_transmission" params="hw_interface:=hardware_interface/EffortJointInterface">
+    <transmission name="arm_01_trans">
+      <type>transmission_interface/SimpleTransmission</type>
+      <joint name="arm_01_joint">
+        <hardwareInterface>${hw_interface}</hardwareInterface>
+      </joint>
+      <actuator name="arm_01Motor">
+        <hardwareInterface>${hw_interface}</hardwareInterface>
+        <mechanicalReduction>1</mechanicalReduction>
+      </actuator>
+    </transmission>
+    <transmission name="arm_02_trans">
+      <type>transmission_interface/SimpleTransmission</type>
+      <joint name="arm_02_joint">
+        <hardwareInterface>${hw_interface}</hardwareInterface>
+      </joint>
+      <actuator name="arm_02Motor">
+        <hardwareInterface>${hw_interface}</hardwareInterface>
+        <mechanicalReduction>1</mechanicalReduction>
+      </actuator>
+    </transmission>
+    <transmission name="arm_03_trans">
+      <type>transmission_interface/SimpleTransmission</type>
+      <joint name="arm_03_joint">
+        <hardwareInterface>${hw_interface}</hardwareInterface>
+      </joint>
+      <actuator name="arm_03Motor">
+        <hardwareInterface>${hw_interface}</hardwareInterface>
+        <mechanicalReduction>1</mechanicalReduction>
+      </actuator>
+    </transmission>
+    <transmission name="arm_04_trans">
+      <type>transmission_interface/SimpleTransmission</type>
+      <joint name="arm_04_joint">
+        <hardwareInterface>${hw_interface}</hardwareInterface>
+      </joint>
+      <actuator name="arm_04Motor">
+        <hardwareInterface>${hw_interface}</hardwareInterface>
+        <mechanicalReduction>1</mechanicalReduction>
+      </actuator>
+    </transmission>
     <transmission name="arm_tools_trans">
       <type>transmission_interface/SimpleTransmission</type>
       <joint name="arm_tools_joint">
-        <hardwareInterface>hardware_interface/EffortJointInterface</hardwareInterface>
+        <hardwareInterface>${hw_interface}</hardwareInterface>
       </joint>
       <actuator name="arm_toolsMotor">
-        <hardwareInterface>hardware_interface/EffortJointInterface</hardwareInterface>
+        <hardwareInterface>${hw_interface}</hardwareInterface>
         <mechanicalReduction>1</mechanicalReduction>
       </actuator>

File: models/curiosity_path/urdf/sensor_mast.xacro (robot description, xacro)
@@ -60,14 +60,4 @@
         <dynamics damping="0.0" friction="0.0"/>
 	</joint>
-    <transmission name="mast_p_trans">
-      <type>transmission_interface/SimpleTransmission</type>
-      <joint name="mast_p_joint">
-        <hardwareInterface>hardware_interface/EffortJointInterface</hardwareInterface>
-      </joint>
-      <actuator name="mast_pMotor">
-        <hardwareInterface>hardware_interface/EffortJointInterface</hardwareInterface>
-        <mechanicalReduction>1</mechanicalReduction>
-      </actuator>
-    </transmission>
   	<link name='mast_p_to_mast_02'>
 		<inertial>
@@ -128,14 +118,4 @@
         <dynamics damping="0.0" friction="0.0"/>
 	</joint>
-    <transmission name="mast_02_trans">
-      <type>transmission_interface/SimpleTransmission</type>
-      <joint name="mast_02_joint">
-        <hardwareInterface>hardware_interface/EffortJointInterface</hardwareInterface>
-      </joint>
-      <actuator name="mast_02Motor">
-        <hardwareInterface>hardware_interface/EffortJointInterface</hardwareInterface>
-        <mechanicalReduction>1</mechanicalReduction>
-      </actuator>
-    </transmission>
 	<link name='mast_02_to_mast_cameras'>
 		<inertial>
@@ -196,14 +176,4 @@
         <dynamics damping="0.0" friction="0.0"/>
 	</joint>
-    <transmission name="mast_02_trans">
-      <type>transmission_interface/SimpleTransmission</type>
-      <joint name="mast_cameras_joint">
-        <hardwareInterface>hardware_interface/EffortJointInterface</hardwareInterface>
-      </joint>
-      <actuator name="mast_02Motor">
-        <hardwareInterface>hardware_interface/EffortJointInterface</hardwareInterface>
-        <mechanicalReduction>1</mechanicalReduction>
-      </actuator>
-    </transmission>
   	<material name="green">
         <color rgba="0 0.8 0 1"/>
@@ -256,3 +226,36 @@
     </joint>
   </xacro:macro>
+  <!-- ros2_control transmission does NOT use this currently. This macro is not actively used -->
+  <xacro:macro name="mast_transmission" params="hw_interface:=hardware_interface/EffortJointInterface">
+    <transmission name="mast_p_trans">
+      <type>transmission_interface/SimpleTransmission</type>
+      <joint name="mast_p_joint">
+        <hardwareInterface>${hw_interface}</hardwareInterface>
+      </joint>
+      <actuator name="mast_pMotor">
+        <hardwareInterface>${hw_interface}</hardwareInterface>
+        <mechanicalReduction>1</mechanicalReduction>
+      </actuator>
+    </transmission>
+    <transmission name="mast_02_trans">
+      <type>transmission_interface/SimpleTransmission</type>
+      <joint name="mast_02_joint">
+        <hardwareInterface>${hw_interface}</hardwareInterface>
+      </joint>
+      <actuator name="mast_02Motor">
+        <hardwareInterface>${hw_interface}</hardwareInterface>
+        <mechanicalReduction>1</mechanicalReduction>
+      </actuator>
+    </transmission>
+    <transmission name="mast_02_trans">
+      <type>transmission_interface/SimpleTransmission</type>
+      <joint name="mast_cameras_joint">
+        <hardwareInterface>${hw_interface}</hardwareInterface>
+      </joint>
+      <actuator name="mast_02Motor">
+        <hardwareInterface>${hw_interface}</hardwareInterface>
+        <mechanicalReduction>1</mechanicalReduction>
+      </actuator>
+    </transmission>
+</xacro:macro>
 </robot>

Commit message: Fix a spacing issue

File: models/curiosity_path/urdf/arm.xacro (robot description, xacro)
@@ -28,8 +28,8 @@
 	<link name='arm_01'>
 		<collision>
-		    <origin xyz="0 0 0" rpy="0 0 0"/>
-		    <geometry>
-		        <mesh filename="package://simulation/models/curiosity_path/meshes/arm_01_fixed.dae" scale="${scale_XYZ} ${scale_XYZ} ${scale_XYZ}"/>
-		    </geometry>
+		        <origin xyz="0 0 0" rpy="0 0 0"/>
+		        <geometry>
+		            <mesh filename="package://simulation/models/curiosity_path/meshes/arm_01_fixed.dae" scale="${scale_XYZ} ${scale_XYZ} ${scale_XYZ}"/>
+		        </geometry>
 		</collision>
 		<visual>
@@ -231,21 +231,21 @@
 	</joint>
   	<link name='arm_04_to_arm_tools'>
-	<inertial>
-            <origin xyz="0 0 0" rpy="0 0 0"/>
-            <mass value="0.02" />
-            <inertia ixx="2.61666666667e-05" ixy="0.0" ixz="0.0" iyy="2.61666666667e-05" iyz="0.0" izz="3.6e-05"/>
-        </inertial>
-        <collision>
-            <origin rpy="0 0 0" xyz="0 0 0"/>
-            <geometry>
-                <cylinder radius="0.02" length="0.02"/>
-            </geometry>
-        </collision>
-		<visual>
-            <origin rpy="0 0 0" xyz="0 0 0"/>
-            <geometry>
-                <cylinder radius="0.02" length="0.02"/>
-            </geometry>
-        </visual>
+	    <inertial>
+                <origin xyz="0 0 0" rpy="0 0 0"/>
+                <mass value="0.02" />
+                <inertia ixx="2.61666666667e-05" ixy="0.0" ixz="0.0" iyy="2.61666666667e-05" iyz="0.0" izz="3.6e-05"/>
+            </inertial>
+            <collision>
+                <origin rpy="0 0 0" xyz="0 0 0"/>
+                <geometry>
+                    <cylinder radius="0.02" length="0.02"/>
+                </geometry>
+            </collision>
+	    <visual>
+                <origin rpy="0 0 0" xyz="0 0 0"/>
+                <geometry>
+                    <cylinder radius="0.02" length="0.02"/>
+                </geometry>
+            </visual>
 	</link>
   	<joint name="arm_04_to_arm_tools_joint" type="fixed">
